File: hardware/keykeyv2.1/keykeyv2.1_r.kicad_pcb (KiCad board)
At the start: 2 copper layers, 158.4 x 122.6 mm, 66 parts, among them J1 AudioJack4(PJ-320A), SW1 SW_Push, SW10 SW_Push, SW11 SW_Push, SW12 SW_Push, SW13 SW_Push, SW14 SW_Push, SW15 SW_Push, SW16 SW_Push, SW17 SW_Push, SW18 SW_Push, SW19 SW_Push, SW2 SW_Push, SW20 SW_Push, SW21 SW_Push, SW22 SW_Push, SW23 SW_Push, SW24 SW_Push, SW25 SW_Push, SW26 SW_Push, SW27 SW_Push, SW28 SW_Push, SW29 SW_Push, SW3 SW_Push, SW30 SW_Push, SW4 SW_Push, SW5 SW_Push, SW6 SW_Push, SW7 SW_Push, SW8 SW_Push, SW9 SW_Push, U2 5way-navigation-switch

Commit message: 업데이트
Connections:
- J1 pad 2: unconnected-(J1-Pad2) -> unconnected-(U1-GP26-Pad26)
Routing:
- net unconnected-(U1-GP26-Pad26): track 0.00 -> 31.4 mm, vias 0 -> 2
